Commit message: fixed mesh dependencies

File: urdf/anymal.urdf (robot description, URDF)
Before this commit: robot anymal, 96 links, 95 joints
Links:
- link LF_FOOT: geometry collision cylinder length=0.39572 radius=0.0175; collision sphere radius=0.031455
- link LF_HAA_drive: geometry visual mesh filename=package://anymal_wbc/meshes/drive.dae scale=1.0 1.0 1.0
- link LF_HFE_drive: geometry collision cylinder length=0.119 radius=0.05375; visual mesh filename=package://anymal_wbc/meshes/drive.dae scale=1.0 1.0 1.0
- link LF_KFE_drive: geometry collision cylinder length=0.119 radius=0.05375; visual mesh filename=package://anymal_wbc/meshes/drive.dae scale=1.0 1.0 1.0
- link LF_hip_fixed: geometry visual mesh filename=package://anymal_wbc/meshes/hip.dae scale=1.0 1.0 1.0
- link LF_shank_fixed: geometry collision box size=0.13283 0.08302 0.05732; collision cylinder length=0.05732 radius=0.071
- link LF_thigh_fixed: geometry collision box size=0.093 0.063 0.285; collision cylinder length=0.08313000000000001 radius=0.07
- link LH_FOOT: geometry collision cylinder length=0.39572 radius=0.0175; collision sphere radius=0.031455
- link LH_HAA_drive: geometry visual mesh filename=package://anymal_wbc/meshes/drive.dae scale=1.0 1.0 1.0
- link LH_HFE_drive: geometry collision cylinder length=0.119 radius=0.05375; visual mesh filename=package://anymal_wbc/meshes/drive.dae scale=1.0 1.0 1.0
- link LH_KFE_drive: geometry collision cylinder length=0.119 radius=0.05375; visual mesh filename=package://anymal_wbc/meshes/drive.dae scale=1.0 1.0 1.0
- link LH_hip_fixed: geometry visual mesh filename=package://anymal_wbc/meshes/hip.dae scale=1.0 1.0 1.0
- link LH_shank_fixed: geometry collision box size=0.13283 0.08302 0.05732; collision cylinder length=0.05732 radius=0.071
- link LH_thigh_fixed: geometry collision box size=0.093 0.063 0.285; collision cylinder length=0.08313000000000001 radius=0.07
- link RF_FOOT: geometry collision cylinder length=0.39572 radius=0.0175; collision sphere radius=0.031455
- link RF_HAA_drive: geometry visual mesh filename=package://anymal_wbc/meshes/drive.dae scale=1.0 1.0 1.0
- link RF_HFE_drive: geometry collision cylinder length=0.119 radius=0.05375; visual mesh filename=package://anymal_wbc/meshes/drive.dae scale=1.0 1.0 1.0
- link RF_KFE_drive: geometry collision cylinder length=0.119 radius=0.05375; visual mesh filename=package://anymal_wbc/meshes/drive.dae scale=1.0 1.0 1.0
- link RF_hip_fixed: geometry visual mesh filename=package://anymal_wbc/meshes/hip.dae scale=1.0 1.0 1.0
- link RF_shank_fixed: geometry collision box size=0.13283 0.08302 0.05732; collision cylinder length=0.05732 radius=0.071
- link RF_thigh_fixed: geometry collision box size=0.093 0.063 0.285; collision cylinder length=0.08313000000000001 radius=0.07
- link RH_FOOT: geometry collision cylinder length=0.39572 radius=0.0175; collision sphere radius=0.031455
- link RH_HAA_drive: geometry visual mesh filename=package://anymal_wbc/meshes/drive.dae scale=1.0 1.0 1.0
- link RH_HFE_drive: geometry collision cylinder length=0.119 radius=0.05375; visual mesh filename=package://anymal_wbc/meshes/drive.dae scale=1.0 1.0 1.0
- link RH_KFE_drive: geometry collision cylinder length=0.119 radius=0.05375; visual mesh filename=package://anymal_wbc/meshes/drive.dae scale=1.0 1.0 1.0
- link RH_hip_fixed: geometry visual mesh filename=package://anymal_wbc/meshes/hip.dae scale=1.0 1.0 1.0
- link RH_shank_fixed: geometry collision box size=0.13283 0.08302 0.05732; collision cylinder length=0.05732 radius=0.071
- link RH_thigh_fixed: geometry collision box size=0.093 0.063 0.285; collision cylinder length=0.08313000000000001 radius=0.07
- link base: geometry collision box size=0.894 0.1615 0.256; collision cylinder length=0.1482 radius=0.089
- link battery: geometry visual mesh filename=package://anymal_wbc/meshes/battery.dae scale=1.0 1.0 1.0
- link bottom_shell: geometry visual mesh filename=package://anymal_wbc/meshes/bottom_shell.dae scale=1.0 1.0 1.0
- link docking_socket: geometry visual mesh filename=package://anymal_wbc/meshes/docking_socket.dae scale=1.0 1.0 1.0
- link face_shell_front: geometry visual mesh filename=package://anymal_wbc/meshes/face_shell.dae scale=1.0 1.0 1.0
- link face_shell_rear: geometry visual mesh filename=package://anymal_wbc/meshes/face_shell.dae scale=1.0 1.0 1.0
- link inspection_payload_mount: geometry collision box size=0.16 0.135 0.015; visual mesh filename=package://anymal_wbc/meshes/mount.dae scale=1 1 1
- link inspection_payload_pan: geometry collision box size=0.18 0.24 0.21; visual mesh filename=package://anymal_wbc/meshes/pan.dae scale=1 1 1
- link inspection_payload_tilt: geometry visual mesh filename=package://anymal_wbc/meshes/tilt.dae scale=1 1 1
- link lidar: geometry collision cylinder length=0.1355 radius=0.07; visual mesh filename=package://anymal_wbc/meshes/lidar.dae
- link top_shell: geometry visual mesh filename=package://anymal_wbc/meshes/top_shell.dae scale=1.0 1.0 1.0

Commit message: removed inspection payload from anymal urdf

File: urdf/anymal.urdf (robot description, URDF)
Before this commit: robot anymal, 96 links, 95 joints
Links:
- removed link inspection_payload_camera
- removed link inspection_payload_camera_default
- removed link inspection_payload_head
- removed link inspection_payload_light
- removed link inspection_payload_microphone
- removed link inspection_payload_mount
- removed link inspection_payload_pan
- removed link inspection_payload_thermal_camera
- removed link inspection_payload_tilt
- added link hatch, mass 0.09653; visual mesh filename=package://anymal_wbc/meshes/hatch.dae scale=1.0 1.0 1.0
Joints:
- removed joint base_to_inspection_payload_mount
- removed joint inspection_payload_head_to_camera
- removed joint inspection_payload_head_to_light
- removed joint inspection_payload_head_to_microphone
- removed joint inspection_payload_head_to_thermal_camera
- removed joint inspection_payload_mount_to_camera_default
- removed joint inspection_payload_mount_to_pan
- removed joint inspection_payload_pan_to_tilt
- removed joint inspection_payload_tilt_to_head
- added joint base_to_hatch: type fixed, parent base, child hatch, origin xyz=0.14253 0.0 0.092 rpy=0 0 0
